File: MegaDrive.kicad_sch (KiCad schematic)
At the start: 171 parts, among them J1 Video, J10 Conn_01x04_Pin, J11 Conn_01x02_Pin, J110 Conn_01x04_Pin, J111 Conn_01x02_Socket, J2 Floppy, J3 Cartridge, J4 EXT, J5 Player1, J6 Player2, J7 Jack-DC, J9 AudioJack3, SW1 SW_SPDT, SW2 SW_Push, U1 68000D, U10 M5M4C264L, U11 YM2612, U12 CXA1034P, U14 LM358, U15 L7805, U17 L7805, U2 uPD42832C-15, U3 uPD42832C-15, U6 Z80CPU, U7 uPD4364, U9 M5M4C264L

Commit message: finalize
Parts:
- added C10, C15, C19, C9: 22pF, Capacitor_SMD:C_0805_2012Metric, symbol Device:C
- added C105, C110, C115, C116, C120, C14, C16, C17, C18, C20, C21, C22, C6, C90: 33pF, Capacitor_SMD:C_0805_2012Metric, symbol Device:C
- added C11, C75, C89: 0,01uF, Capacitor_SMD:C_0805_2012Metric, symbol Device:C
- added C111, C60, C63, C66, CP112: 47uF 10V, Capacitor_THT:CP_Radial_Tantal_D4.5mm_P5.00mm, symbol Device:C_Polarized
- added C112, C92: 33p, Capacitor_SMD:C_0805_2012Metric, symbol Device:C
- added C114: 150pF, Capacitor_SMD:C_0805_2012Metric, symbol Device:C
- added C118, C45: C, Capacitor_SMD:C_0805_2012Metric, symbol Device:C
- added C119, C46, C47, C48, C95: 0.1uF, Capacitor_SMD:C_0805_2012Metric, symbol Device:C
- added C121: 0,1uF, Capacitor_SMD:C_0805_2012Metric, symbol Device:C
- added C33: 0.01u, Capacitor_SMD:C_0805_2012Metric, symbol Device:C
- added C34: 180pF, Capacitor_SMD:C_0805_2012Metric, symbol Device:C
- added C35, C96: 12pF, Capacitor_SMD:C_0805_2012Metric, symbol Device:C
- added C37, C85: 100pF, Capacitor_SMD:C_0805_2012Metric, symbol Device:C
- added C65: 47uF 16V, Capacitor_THT:CP_Radial_Tantal_D4.5mm_P5.00mm, symbol Device:C_Polarized
- added C69, C91, C93: 330pF, Capacitor_SMD:C_0805_2012Metric, symbol Device:C
- added C77: 1000pF, Capacitor_SMD:C_0805_2012Metric, symbol Device:C
- added C78, C88: 47, Capacitor_SMD:C_0805_2012Metric, symbol Device:C
- added C81: 220p, Capacitor_SMD:C_0805_2012Metric, symbol Device:C
- added C82: 20p, Capacitor_SMD:C_0805_2012Metric, symbol Device:C
- added C86: 220uF 10V, Capacitor_THT:CP_Radial_Tantal_D4.5mm_P5.00mm, symbol Device:C_Polarized
- added C87: 0.022u, Capacitor_SMD:C_0805_2012Metric, symbol Device:C
- added H1, H10, H11, H12, H2, H3, H4, H5, H7, H8, H9: MountingHole, MountingHole:MountingHole_3.2mm_M3, symbol Mechanical:MountingHole
- added H6: MountingHole, MountingHole:MountingHole_4mm, symbol Mechanical:MountingHole
- added J9, J99: Conn_01x02_Pin, Connector_PinSocket_2.54mm:PinSocket_1x02_P2.54mm_Vertical, symbol Connector:Conn_01x02_Pin
- added JP5, JP6, JP7: Conn_01x01_Pin, Connector_PinSocket_2.54mm:PinSocket_1x01_P2.54mm_Vertical, symbol Connector:Conn_01x01_Pin
- added L2, L3, L7: 100mH, Resistor_THT:R_Axial_DIN0204_L3.6mm_D1.6mm_P5.08mm_Horizontal, symbol Device:L
- added L5: 12mH, Resistor_THT:R_Axial_DIN0204_L3.6mm_D1.6mm_P5.08mm_Horizontal, symbol Device:L
- added R10, R11, R12, R14, R15, R16, R71, R8, R9: 2.2k, Resistor_SMD:R_0805_2012Metric, symbol Device:R
- added R13, R33, R50: 75, Resistor_SMD:R_0805_2012Metric, symbol Device:R
- added R26, R29, R69: 1k, Resistor_SMD:R_0805_2012Metric, symbol Device:R
- added R27, R28, R67: 1.2k, Resistor_SMD:R_0805_2012Metric, symbol Device:R
- added R3: 120, Resistor_SMD:R_0805_2012Metric, symbol Device:R
- added R30: 24k, Resistor_SMD:R_0805_2012Metric, symbol Device:R
- added R36, R39, R49, R52: R, Resistor_SMD:R_0805_2012Metric, symbol Device:R
- added R59, R77, R78, R79, R80, R81, R82, R83, R84: 4.7k, Resistor_SMD:R_0805_2012Metric, symbol Device:R
- added R64: 10k, Resistor_SMD:R_0805_2012Metric, symbol Device:R
- added R65: 100k, Resistor_SMD:R_0805_2012Metric, symbol Device:R
- added R68: 220, Resistor_SMD:R_0805_2012Metric, symbol Device:R
- added R70: 2k, Resistor_SMD:R_0805_2012Metric, symbol Device:R
- added R72: 1.3k, Resistor_SMD:R_0805_2012Metric, symbol Device:R
- added R74: 33k, Resistor_SMD:R_0805_2012Metric, symbol Device:R
- added R85: 10, Resistor_SMD:R_0805_2012Metric, symbol Device:R
- C117, C122, C39, C80, C94: now not fitted; now left out of the parts list
- C59: value ~ -> 47uF 10V
- C68: renamed from C86; value 100uF 10V -> 47uF 10V; footprint Capacitor_THT:CP_Radial_D8.0mm_P5.00mm -> Capacitor_THT:CP_Radial_Tantal_D4.5mm_P5.00mm
- C74, C79: footprint Capacitor_THT:CP_Radial_D8.0mm_P5.00mm -> Capacitor_THT:CP_Radial_Tantal_D4.5mm_P5.00mm
- D2: value D -> 1S2475
- FB1, FB10, FB13, FB14, FB2, FB3, FB4, FB5, FB8, FB9: footprint Ferrite_THT:LairdTech_28C0236-0JW-10 -> Inductor_THT:L_Axial_L7.0mm_D3.3mm_P5.08mm_Vertical_Fastron_MICC
- J7: footprint Connector:JWT_A3963_1x02_P3.96mm_Vertical -> SEGA:DCJack
- J8: renamed from J9; footprint Connector_Audio:Jack_3.5mm_CUI_SJ1-3523N_Horizontal -> SEGA:Jack_3.5mm
- RV1: footprint (none) -> SEGA:HeadphoneVolumeSlider
Connections:
- net DTACK is gone; now on net ~{DTAK}: U1.10 (DTACK), U4.129 (~{DTAK})
- net +9VA: now also C89.1, C91.1
- net BGACK: now also R11.1
- net BR: now also R12.1
- net GND: now also FB2.2, RV1.1, U8.48 (SEL1), C10.2, C105.2, C11.2, C110.2, C111.2, C112.1, C114.2, C115.2, C116.2, C118.2, C119.2, C120.2, C121.2, C14.2, C15.2, C16.2, C17.2, C18.2, C19.2, C20.2, C21.2, C22.2, C34.2, C37.2, C6.2, C60.2, C63.2, C65.2, C66.2, C69.1, C75.2, C77.1, C78.2, C81.1, C82.2, C85.1, C88.2, C89.2, C9.2, C90.2, C91.2, C92.1, C93.2, C95.2, CP112.2, J9.2 (Pin_2), J99.2 (Pin_2), L5.1, R13.1, R26.1, R30.1, R33.1, R49.1, R50.1, R71.1; no longer FB2.1, R51.2, RV1.3
- net IPL1: now also R10.1
- net IPL2: now also R9.1
- net NTSC: now also JP3.1 (A), JP4.1 (A), U13.7 (NTSC/PAL), U4.154 (NTSC)
- net VA1: now also C90.1
- net VA21: now also C81.2
- net VA7: now also C120.1
- net VCC: now also C18.1, C19.1, C20.1, C21.1, C6.1, C65.1, C66.1, R10.2, R11.2, R12.2, R14.2, R15.2, R16.1, R68.2, R69.2, R8.2, R9.2
- net VCCQ: now also C24.1, D2.1 (K), L6.1, R55.1, R56.1, R57.1, U13.12 (Vcc1), U13.19 (Vcc2), U8.30 (AVC), C10.1, C111.1, C14.1, C15.1, C16.1, C22.1, C63.1, C9.1, CP112.1, L2.1, R3.1, R59.1, R67.2, R77.1, R78.1, R79.1, R80.1, R81.1, R82.1, R83.1, R84.1; no longer D2.2 (A)
- net VDDA: now also C23.1, U11.22 (AVcc), U14.8 (V+), U8.94 (AYS), C17.1, C60.1, C69.2, L2.2; no longer R55.1, R56.1, R57.1
- net ZA0: now also R59.2
- net ZD0: now also R77.2
- net ZD1: now also R78.2
- net ZD2: now also R79.2
- net ZD3: now also R80.2
- net ZD4: now also R81.2
- net ZD5: now also R82.2
- net ZD6: now also R83.2
- net ZD7: now also R84.2
- net ~{ASEL}: now also J2.a22 (Pin_a22), U4.108
- net ~{AS}: now also R68.1
- net ~{CART}: now also C119.1
- net ~{CAS0}: now also J2.a3 (Pin_a3), J3.b16 (Pin_b16), U4.113
- net ~{M3}: now also U8.45 (SEL0), C77.2
- net ~{RAS0}: now also JP5.1 (Pin_1)
- net ~{SRES}: now also U14.7, C118.1, C85.2, R65.2
- net ~{TIME}: now also U4.109 (~{TIME})
- net ~{UWR}: now also U3.27 (~{WE})
- net ~{VRES}: now also U1.18 (RESET), U4.134 (~{VRES})
- net at C61.1: now also R51.2
- net SL2: now reaches C61.2
- net SL2: now also J2.b29 (Pin_b29), R50.2
- net at C42.1: now also R36.2
- net SL1: now reaches C42.2
- net SL1: now also J3.b1 (Pin_b1), R13.2
- net at R35.2, R40.1: now also R34.2, R51.1, U12.2 (EQ_IN_(A)), C45.1, C46.1, R36.1
- net at R40.2, R42.2, U12.1 (EQ_OUT_(A)): now also C45.2
- net at C62.1: now also R52.1
- net SR2: now reaches C62.2
- net SR2: now also J2.a29 (Pin_a29), R49.2
- net ~{VDPM}: now reaches U8.102 (~{MREQ})
- net ~{VDPM}: now also U4.106 (~{VDPM})
- net ~{INTAK}: now reaches U8.103 (~{INTAK})
- net ~{INTAK}: now also U4.157 (~{INTAR})
- net ~{IREQ}: now reaches U8.106 (~{IORQ})
- net ~{IREQ}: now also U4.13 (~{TREQ}), U6.20 (~{IORQ})
- net ~{ZRD}: now reaches U8.107 (~{RD})
- net ~{ZRD}: now also U11.16 (RD), U4.12 (~{ERD}), U6.21 (~{RD}), U7.22 (~{OE})
- net ~{ZWR}: now reaches U8.108 (~{WR})
- net ~{ZWR}: now also U11.15 (WR), U4.11 (~{EWR}), U6.22 (~{WR}), U7.27 (~{WE})
- net ~{M1}: now reaches U8.109 (~{M1})
- net ~{M1}: now also U4.6 (~{MI}), U6.27 (~{M1})
- net ~{DTAK}: now reaches U8.114 (~{DTAK})
- net ~{DTAK}: now also J3.b20 (Pin_b20), R8.1
- net ~{OE0}: now reaches U8.117 (~{OE0})
- net ~{OE0}: now also U4.112 (~{OE0})
- net ~{YS}: now reaches U8.39 (~{YS})
- net ~{YS}: now also J3.b12 (Pin_b12), C110.1
- net at U8.40 (SPA/B): now also R14.1
- net ~{VSYNC}: now reaches U8.41 (~{VSYNC})
- net ~{VSYNC}: now also J3.b13 (Pin_b13), C115.1
- net ~{HSYNC}: now reaches U8.43 (~{HSYNC})
- net ~{HSYNC}: now also J3.b14 (Pin_b14), U4.155 (~{HSYNC}), C116.1, R67.1
- net ~{HL}: now reaches U8.44 (~{HL})
- net ~{HL}: now also U4.101
- net at U8.49 (CLK1): now also C78.1
- net at U8.51 (CLK0): now also C88.1
- net EDCK: now reaches U8.53 (EDCK)
- net EDCK: now also FB7.1, J3.b15 (Pin_b15), C112.2
- net at C39.1, C40.2, U8.95 (SOUND): no longer R51.1
- net ~{INT}: now reaches U8.98 (~{INT})
- net ~{INT}: now also U6.16 (~{INT}), R15.1
- net ~{ZBAK}: now reaches U4.10 (~{ZBAR})
- net ~{ZBAK}: now also U6.23 (~{BUSACK})
- net ~{FDHR}: now reaches U4.102
- net ~{FDHR}: now also J2.b24 (Pin_b24)
- net ~{FDC}: now reaches U4.103
- net ~{FDC}: now also J2.a24 (Pin_a24)
- net FRES: now reaches U4.105 (FRES)
- net FRES: now also J2.a25 (Pin_a25)
- net ~{ROM}: now reaches U4.107 (~{ROM})
- net ~{ROM}: now also J2.a21 (Pin_a21)
- net ~{RAS2}: now reaches U4.110 (~{RAS2})
- net ~{RAS2}: now also J2.a23 (Pin_a23)
- net ~{CAS2}: now reaches U4.111 (~{CAS2})
- net ~{CAS2}: now also J2.b23 (Pin_b23), J3.b21 (Pin_b21), C93.1
- net ~{NOE}: now reaches U4.118 (~{NOE})
- net ~{NOE}: now also U2.22 (~{OE}), JP6.1 (Pin_1)
- net ~{EOE}: now reaches U4.119 (~{EOE})
- net ~{EOE}: now also C117.1, U3.22 (~{OE}), JP7.1 (Pin_1)
- net VCLK: now reaches U1.15 (CLK), U4.123 (VCLK)
- net VCLK: now also J3.b19 (Pin_b19), U11.24 (CLOCK_IN)
- net ~{MREQ}: now reaches U4.14 (~{MREQ})
- net ~{MREQ}: now also U6.19 (~{MREQ})
- net ~{NMI}: now reaches U4.15 (~{NMI}), U6.17 (~{NMI})
- net ~{SOUND}: now reaches U4.156 (~{SOUND})
- net ~{SOUND}: now also U11.14 (CS)
- net at U4.158 (EDCK): now also R85.1
- net ~{ZRAM}: now reaches U4.4 (~{ZRAM})
- net ~{ZRAM}: now also U7.20 (~{CE1}), C114.1
- net ~{REF}: now reaches U4.5 (~{RAF})
- net ~{REF}: now also U7.1 (~{RFSH})
- net ~{JAP}: now reaches JP1.1 (A), JP2.1 (A), U4.72 (~{JAP})
- net at U4.9 (~{WAIT}): now also U6.24 (~{WAIT})
- net at FB13.1: now also RF1.2 (VIDEO)
- net at FB13.2: now also C86.2, R71.2; no longer RF1.2 (VIDEO)
- net at FB9.1: now also J1.3; no longer C32.1
- net at FB9.2: now also C32.1; no longer J1.3
- net DCin1: now reaches J111.1 (Pin_1), J7.1
- net DCin2: now reaches J111.2 (Pin_2), J7.2
- net at J11.1 (Pin_1): now also FB1.1; no longer FB1.2
- net at J11.2 (Pin_2): now also FB2.1; no longer FB2.2
- net at FB14.1, R73.2: now also C87.1, R72.2
- net at R58.1, R66.1: now also RV1.3; no longer RV1.1
- net at U13.13 (I_REF): now also C95.1, R30.2
- net VREF: now reaches U13.14 (V_REF)
- net VREF: now also C38.1, U14.6 (-), R29.1
- net at U13.15 (CHROMA_OUT): now also R28.1
- net at U13.16 (Y_OUT): now also R27.1
- net at U13.17 (CHROMA_IN): now also C33.1
- net at U13.18 (Y_IN): now also C34.1, C35.1, L3.2, R29.2
- net at R25.2, U13.20 (C_VIDEO_OUT): now also R70.2
- net at C31.2, U13.9 (AUDIO_OUT): now also C87.2, R72.1
- net at R42.1, R43.1, U14.2 (-): now also R74.1
- net at C51.1, U12.11 (OUT_(B)): now also C11.1
- net at C50.1, U12.14 (OUT_(A)): now also C75.1
- net at C49.1, R58.2, U12.3 (IN_(A))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: now also C46.2, C47.2
- net at R37.2, U12.7 (EQ_IN_(B)): now also R38.2, R41.1, C47.1, C48.1, R39.2, R52.2
- net at R41.2, R43.2, U12.8 (EQ_OUT_(B)): now also C48.2
- net at FB6.1, OSC1.8 (OUT): now also C82.1, R69.1
- net at C30.2, U14.1: now also R74.2
- net at U14.5 (+): now also R64.2, R65.1
- net ~{MRES}: now reaches C64.1, R1.2
- net ~{MRES}: now also D2.2 (A), J3.b2 (Pin_b2), R64.1; no longer D2.1 (K)
- net at FB7.2: now also C92.2, R85.2
- net at SW1.2 (B): now also FB1.2, C121.1; no longer FB1.1
- net at C44.1: now also R39.1
- net SR1: now reaches C44.2
- net SR1: now also J3.b3 (Pin_b3), R33.2
- net at C40.1, R37.1: now also R34.1
- net ~{CSYNC}: no longer names the net of C103.1, C113.1, J1.7, U13.10 (C_SYNC_IN), U8.42 (~{CSYNC})
- net ~{CSYNC}: now also C105.1, R16.2
- new net: C96.1, L7.1
- new net: C37.1, C96.2, L5.2, R28.2
- new net: C33.2, L7.2, R26.2
- new net: J9.1 (Pin_1), J99.1 (Pin_1), R3.2
- new net: C35.2, L3.1, R27.2
- new net: C86.1, R70.1
- no-connect marks 11 -> 34
Other:
- moved on the sheet: C13, C23, C38, C42, C44, C5, C51, C52, C59, C61, C62, C64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
